Commit message: added table

File: arm_actions/urdf/gen3.urdf (robot description, URDF)
Before this commit: robot gen3_robotiq_2f_85, 13 links, 12 joints
Links:
- added link table; collision box size=2 2 0.1; visual box size=2 2 0.1
Joints:
- added joint arm_table_joint: type fixed, parent table, child base_link, origin xyz=0 0 0.1 rpy=0 0 0
